Commit message: modify

File: urdf/satellite.urdf (robot description, URDF)
Before this commit: robot satellite, 2 links, 1 joints
Links:
- link satellite: geometry visual mesh filename=package://point/meshes/satellite0.01.stl

Commit message: modify package name

File: urdf/satellite.urdf (robot description, URDF)
Before this commit: robot satellite, 2 links, 1 joints
Links:
- link satellite: geometry visual mesh filename=package://ros-slam/meshes/satellite0.01.stl
